File: kicad/nerf.sch (KiCad schematic (older format))
At the start: 20 parts

Commit message: new proto board adapting
Parts:
- removed P? (x2): CONN_01X02, symbol CONN_01X02
- removed P?: CONN_01X05, symbol CONN_01X05
- removed P?: CONN_01X04, symbol CONN_01X04
- removed P? (x3): CONN_01X03, symbol CONN_01X03
- added P?: CONN_02X05, symbol CONN_02X05
- added P?: CONN_02X07, symbol CONN_02X07
- U2: renamed from U?; symbol ULN2003 -> ULN2003-RESCUE-nerf
- gave numbers to parts that had none: 11
Connections:
- net +3V3: now also P?.3 (P3), P?.8 (P8)
- net +BATT: now also P?.9 (P9)
- net GND: now also P?.1 (P1), P?.11 (P11), P?.12 (P12), P?.4 (P4), P?.5 (P5)
- net at U2.13 (O4): now also P?.7 (P7)
- net at U2.14 (O3): now also P?.5 (P5)
- net at U2.15 (O2): now also P?.6 (P6)
- net at U2.16 (O1): now also P?.4 (P4)
- net at K1.12 (C2): now also P?.9 (P9)
- net at K1.16 (T2): now also P?.10 (P10)
- net at X1.1 (P0.6): now also P?.1 (P1)
- net at X1.12 (P2.11): now also P?.10 (P10)
- net at X1.15 (P0.0): now also P?.7 (P7)
- net at X1.16 (P0.5): now also P?.8 (P8)
- net at X1.2 (P0.7): now also P?.2 (P2)
- net at X1.3 (P0.8): now also P?.3 (P3)
- net at X1.7 (P2.0): now also P?.6 (P6)
- net at X1.8 (P2.6): now also P?.2 (P2)
- net at R3.2, U1.3 (+): now also P?.14 (P14)
- net at R4.2, U1.5 (+): now also P?.13 (P13)
